File: PCB GUIDANCE/PCB GUIDANCE.kicad_sch (KiCad schematic)
At the start: 24 parts, among them SW1 SW_Push, U1 ATmega32U4-A, Y1 16MHz

Commit message: big
Parts:
- added D5, D6, D7, D8: D_Small, Diode_SMD:D_SOD-123, symbol Device:D_Small
- added MX5, MX6, MX7, MX8: MX-NoLED, MX_Alps_Hybrid:MX-1U, symbol MX_Alps_Hybrid:MX-NoLED
Connections:
- net COL1: now also MX5.1 (COL), MX6.1 (COL), MX7.1 (COL), MX8.1 (COL)
- net ROW0: now also D5.1 (K), D7.1 (K)
- net ROW1: now also D6.1 (K), D8.1 (K)
- new net: D8.2 (A), MX8.2 (ROW)
- new net: D7.2 (A), MX7.2 (ROW)
- new net: D5.2 (A), MX5.2 (ROW)
- new net: D6.2 (A), MX6.2 (ROW)
