File: PCB GUIDANCE/_autosave-PCB GUIDANCE.kicad_pcb (KiCad board)
At the start: 2 copper layers, 205 x 84.5 mm, 32 parts, among them SW1 SW_Push, U1 ATmega32U4-A, Y1 16MHz

Commit message: big
Parts:
- moved R2 14.7 mm to (54.7, 73.8)
Routing:
- net GND: track 0.00 -> 158.4 mm, vias 0 -> 3
- net +5V: track 0.00 -> 99.7 mm, vias 0 -> 7
- net VCC: track 0.00 -> 68.8 mm
- net Net-(U1-D-): track 0.00 -> 62.4 mm, vias 0 -> 2
- net Net-(U1-D+): track 0.00 -> 53.8 mm, vias 0 -> 2
- net Net-(U1-~{RESET}): track 0.00 -> 50.9 mm
- net unconnected-(U1-PD4-Pad25): track 0.00 -> 47.1 mm, vias 0 -> 1
- net unconnected-(U1-PF1-Pad40): track 0.00 -> 30.0 mm, vias 0 -> 1
- net Net-(U1-UCAP): track 0.00 -> 29.2 mm, vias 0 -> 2
- net unconnected-(U1-PF7-Pad36): track 0.00 -> 29.0 mm, vias 0 -> 1
- net unconnected-(U1-PF6-Pad37): track 0.00 -> 27.6 mm, vias 0 -> 1
- net Net-(U1-XTAL1): track 0.00 -> 18.3 mm
- net Net-(U1-XTAL2): track 0.00 -> 17.4 mm, vias 0 -> 2
- net Net-(U1-~{HWB}/PE2): track 0.00 -> 16.3 mm
- net D+: track 0.00 -> 10.8 mm
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