File: PCB GUIDANCE/PCB GUIDANCE.kicad_pcb (KiCad board)
At the start: 2 copper layers, 205 x 84.5 mm, 32 parts, among them SW1 SW_Push, U1 ATmega32U4-A, Y1 16MHz

Commit message: w
Parts:
- moved R2 14.7 mm to (54.7, 73.8)
Routing:
- net GND: track 0.00 -> 158.4 mm, vias 0 -> 3
- net +5V: track 0.00 -> 99.7 mm, vias 0 -> 7
- net VCC: track 0.00 -> 68.8 mm
- net Net-(U1-D-): track 0.00 -> 62.4 mm, vias 0 -> 2
- net unconnected-(U1-PD6-Pad26): track 0.00 -> 61.8 mm, vias 0 -> 1
- net unconnected-(U1-PC7-Pad32): track 0.00 -> 60.5 mm, vias 0 -> 3
- net Net-(U1-D+): track 0.00 -> 53.8 mm, vias 0 -> 2
- net Net-(U1-~{RESET}): track 0.00 -> 50.9 mm
- net unconnected-(U1-PD4-Pad25): track 0.00 -> 47.1 mm, vias 0 -> 1
- net unconnected-(U1-PF1-Pad40): track 0.00 -> 30.0 mm, vias 0 -> 1
- net Net-(U1-UCAP): track 0.00 -> 29.2 mm, vias 0 -> 2
- net unconnected-(U1-PF7-Pad36): track 0.00 -> 29.0 mm, vias 0 -> 1
- net unconnected-(U1-PB3-Pad11): track 0.00 -> 28.1 mm, vias 0 -> 1
- net unconnected-(U1-PF6-Pad37): track 0.00 -> 27.6 mm, vias 0 -> 1
- net Net-(U1-XTAL1): track 0.00 -> 18.3 mm
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
Commit message: omg big updteate
Parts:
- C1, C2, C3, C4, C5, C6: footprint Capacitor_SMD:C_0805_2012Metric -> Capacitors_SMD:C_0805; moved to B.Cu
- C7: footprint Capacitor_SMD:C_0805_2012Metric -> Capacitors_SMD:C_0805
- F1: footprint Fuse:Fuse_1206_3216Metric -> Fuse_Holders_and_Fuses:Fuse_SMD1206_Reflow; moved to B.Cu
- R1: value R_Small -> 10k; footprint Resistor_SMD:R_0805_2012Metric -> Resistors_SMD:R_0805; moved to B.Cu
- R2, R3, R4: footprint Resistor_SMD:R_0805_2012Metric -> Resistors_SMD:R_0805; moved to B.Cu
- SW1: moved to B.Cu
- U1: value ATmega32U4-A -> ATmega32U4-AU; footprint Package_QFP:TQFP-44_10x10mm_P0.8mm -> Housings_QFP:TQFP-44_10x10mm_Pitch0.8mm; moved to B.Cu
- USB1: footprint random-keyboard-parts:Molex-0548190589 -> random-keyboard-parts:Molex-0548190589-Assembly; moved to B.Cu
- Y1: value 16MHz -> Crystal_GND24_Small; footprint Crystal:Crystal_SMD_3225-4Pin_3.2x2.5mm -> Crystals:Crystal_SMD_3225-4pin_3.2x2.5mm; moved to B.Cu
- moved R4 41.6 mm to (88.2, 124.3)
- moved R2 37.5 mm to (60.9, 110.7)
- moved R3 36.9 mm to (57.6, 110.7)
- moved F1 29.9 mm to (54.9, 116.2)
- moved SW1 28.9 mm to (58.5, 132.3)
- moved USB1 19.2 mm to (77.9, 65.0)
- moved C4 16.4 mm to (71.4, 110.9), turned to 90 degrees
- moved C3 16.2 mm to (68.7, 118.6), turned to 180 degrees
- moved C2 16.1 mm to (74.3, 106.2), turned to -90 degrees
- moved U1 15.4 mm to (78.9, 119.1), turned to 0 degrees
- moved Y1 15.0 mm to (78.5, 106.2), turned to 180 degrees
- moved R1 13.8 mm to (68.0, 110.9), turned to -90 degrees
- moved C1 13.5 mm to (82.8, 106.2), turned to 90 degrees
- moved C6 13.2 mm to (83.6, 128.3), turned to 180 degrees
- moved C5 11.3 mm to (88.0, 114.4), turned to 90 degrees
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Connections:
- C1 pad 1: GND -> (no net)
- C1 pad 2: Net-(U1-XTAL1) -> GND
- C2 pad 1: GND -> (no net)
- C2 pad 2: Net-(U1-XTAL2) -> GND
- C3 pad 1: Net-(U1-UCAP) -> (no net)
- F1 pad 1: VCC -> +5V
- F1 pad 2: +5V -> VCC
- R1 pad 2: Net-(U1-~{RESET}) -> (no net)
- R2 pad 1: D+ -> (no net)
- R2 pad 2: Net-(U1-D+) -> D+
- R3 pad 1: D- -> (no net)
- R3 pad 2: Net-(U1-D-) -> D-
- R4 pad 1: Net-(U1-~{HWB}/PE2) -> GND
- R4 pad 2: GND -> (no net)
- SW1 pad 2: Net-(U1-~{RESET}) -> (no net)
- U1 pad 1: unconnected-(U1-PE6-Pad1) -> (no net)
- U1 pad 10: unconnected-(U1-PB2-Pad10) -> (no net)
- U1 pad 11: unconnected-(U1-PB3-Pad11) -> (no net)
- U1 pad 12: unconnected-(U1-PB7-Pad12) -> (no net)
- U1 pad 13: Net-(U1-~{RESET}) -> (no net)
- U1 pad 16: Net-(U1-XTAL2) -> (no net)
- U1 pad 17: Net-(U1-XTAL1) -> (no net)
- U1 pad 18: unconnected-(U1-PD0-Pad18) -> (no net)
- U1 pad 19: unconnected-(U1-PD1-Pad19) -> (no net)
- U1 pad 20: unconnected-(U1-PD2-Pad20) -> (no net)
- U1 pad 21: unconnected-(U1-PD3-Pad21) -> (no net)
- U1 pad 22: unconnected-(U1-PD5-Pad22) -> (no net)
- U1 pad 25: unconnected-(U1-PD4-Pad25) -> (no net)
- U1 pad 26: unconnected-(U1-PD6-Pad26) -> (no net)
- U1 pad 27: unconnected-(U1-PD7-Pad27) -> ROW0
- U1 pad 28: unconnected-(U1-PB4-Pad28) -> COL1
- U1 pad 29: unconnected-(U1-PB5-Pad29) -> col
- U1 pad 3: Net-(U1-D-) -> (no net)
- U1 pad 30: unconnected-(U1-PB6-Pad30) -> ROW1
- U1 pad 31: unconnected-(U1-PC6-Pad31) -> (no net)
- U1 pad 32: unconnected-(U1-PC7-Pad32) -> (no net)
- U1 pad 33: Net-(U1-~{HWB}/PE2) -> (no net)
- U1 pad 36: unconnected-(U1-PF7-Pad36) -> (no net)
- U1 pad 37: unconnected-(U1-PF6-Pad37) -> (no net)
- U1 pad 38: unconnected-(U1-PF5-Pad38) -> (no net)
- U1 pad 39: unconnected-(U1-PF4-Pad39) -> (no net)
- U1 pad 4: Net-(U1-D+) -> (no net)
- U1 pad 40: unconnected-(U1-PF1-Pad40) -> (no net)
- U1 pad 41: unconnected-(U1-PF0-Pad41) -> (no net)
- U1 pad 42: unconnected-(U1-AREF-Pad42) -> (no net)
- U1 pad 6: Net-(U1-UCAP) -> (no net)
- U1 pad 8: unconnected-(U1-PB0-Pad8) -> (no net)
- U1 pad 9: unconnected-(U1-PB1-Pad9) -> (no net)
- USB1 pad 2: unconnected-(USB1-ID-Pad2) -> (no net)
- Y1 pad 1: Net-(U1-XTAL1) -> (no net)
- Y1 pad 3: Net-(U1-XTAL2) -> (no net)
Routing:
- net (no net): track 0.00 -> 107.2 mm, vias 0 -> 2
- net ROW1: track 143.8 -> 239.5 mm, vias 0 -> 1
- net Net-(U1-D-): track 62.4 -> 0.00 mm, vias 2 -> 0
- net unconnected-(U1-PD6-Pad26): track 61.8 -> 0.00 mm, vias 1 -> 0
- net unconnected-(U1-PC7-Pad32): track 60.5 -> 0.00 mm, vias 3 -> 0
- net Net-(U1-D+): track 53.8 -> 0.00 mm, vias 2 -> 0
- net Net-(U1-~{RESET}): track 50.9 -> 0.00 mm
- net unconnected-(U1-PD4-Pad25): track 47.1 -> 0.00 mm, vias 1 -> 0
- net D-: track 6.26 -> 48.6 mm
- net COL1: track 175.1 -> 213.3 mm, vias 0 -> 2
- net D+: track 10.8 -> 48.6 mm
- net unconnected-(U1-PF1-Pad40): track 30.0 -> 0.00 mm, vias 1 -> 0
- net Net-(U1-UCAP): track 29.2 -> 0.00 mm, vias 2 -> 0
- net unconnected-(U1-PF7-Pad36): track 29.0 -> 0.00 mm, vias 1 -> 0
- net unconnected-(U1-PB3-Pad11): track 28.1 -> 0.00 mm, vias 1 -> 0
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- added copper zone on B.Cu, net GND
Other:
- board size 205 x 84.5 mm -> 204.9 x 84.6 mm
- board text added: "Imagine clearing Delta you donkey"

Commit message: w
Parts:
- moved D8 32.8 mm to (233.0, 122.7)
- moved MX8 32.8 mm to (216.5, 128.2)
- moved D4 25.1 mm to (221.4, 102.6)
- moved D5 25.1 mm to (241.2, 102.6)
- moved MX4 25.1 mm to (221.6, 88.8)
- moved MX5 25.1 mm to (240.9, 88.8)
- moved MX6 25.1 mm to (260.1, 88.8)
- moved D6 25.1 mm to (260.3, 102.7)
- moved D7 4.86 mm to (123.2, 122.6)
- moved MX7 4.86 mm to (138.7, 128.1)
Routing:
- net ROW1: track 239.5 -> 279.0 mm
- net COL1: track 213.3 -> 248.3 mm
- net ROW0: track 158.9 -> 188.8 mm
- net Net-(D7-A): track 16.5 -> 15.9 mm
Other:
- board outline removed
